File: bottom/bottom.kicad_pcb (KiCad board)
At the start: 2 copper layers, 27.5 x 18.6 mm, 6 parts, among them P1 HLW4R-2C7LF, P2 BP167911-05340H0A

Commit message: Capitalize UGL library name for the board.
Parts:
- removed the ? at (219.3, 149.8)
- removed the ? at (199.8, 149.8)
- removed the ? at (199.8, 136.8)
- added ?: , UGL:hole_2.8mm, F.Cu at (219.3, 149.8)
- added ?: , UGL:hole_2.8mm, F.Cu at (199.8, 149.8)
- added ?: , UGL:hole_2.8mm, F.Cu at (199.8, 136.8)
- G***: footprint ugl:UHK_Logo_12x3.4_mm -> UGL:UHK_Logo_12x3.4_mm
- P1: footprint ugl:HLW4R-2C7LF -> UGL:HLW4R-2C7LF
- P2: footprint ugl:UHK_Male_Pogo_Pin_v2 -> UGL:UHK_Male_Pogo_Pin_v2
Changed lines of the file:
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@@
     (add_net /VCC)
   )
-  (module ugl:hole_2.8mm locked (layer F.Cu)
+  (module UGL:hole_2.8mm locked (layer F.Cu)
     (at 219.35 149.839996)
     (attr virtual)
@@
     (pad "" np_thru_hole circle (at 0 0) (size 2.8 2.8) (drill 2.8) (layers *.Cu *.Mask))
   )
-  (module ugl:hole_2.8mm locked (layer F.Cu)
+  (module UGL:hole_2.8mm locked (layer F.Cu)
     (at 199.85 149.839996)
     (attr virtual)
@@
     (pad "" np_thru_hole circle (at 0 0) (size 2.8 2.8) (drill 2.8) (layers *.Cu *.Mask))
   )
-  (module ugl:hole_2.8mm locked (layer F.Cu)
+  (module UGL:hole_2.8mm locked (layer F.Cu)
     (at 199.85 136.839997)
     (attr virtual)
@@
     (pad "" np_thru_hole circle (at 0 0) (size 2.8 2.8) (drill 2.8) (layers *.Cu *.Mask))
   )
-  (module ugl:UHK_Logo_12x3.4_mm (layer B.Cu)
+  (module UGL:UHK_Logo_12x3.4_mm (layer B.Cu)
     (at 209.6 149.7 180)
     (attr virtual)
@@
       (xy 2.528295 1.556775)) (layer B.Mask) (width 0.01))
   )
-  (module ugl:HLW4R-2C7LF locked (layer F.Cu)
+  (module UGL:HLW4R-2C7LF locked (layer F.Cu)
     (at 207.85 143.04 270)
     (descr "FFC connector")
@@
       (net 4 /GND))
   )
-  (module ugl:UHK_Male_Pogo_Pin_v2 locked (layer F.Cu)
+  (module UGL:UHK_Male_Pogo_Pin_v2 locked (layer F.Cu)
     (at 225.35 143.139999)
     (fp_text reference P2 (at -2.95 8.360001) (layer F.SilkS)
