File: top/touchpad-top.kicad_pcb (KiCad board)
At the start: 2 copper layers, 28.3 x 40 mm, 142 parts, among them P1 CONN_10, P2 CONN_5, U1 IQS572, U4 ESD

Commit message: Final version.
Parts:
- R1: value 0 -> 33; footprint UGL:SM0603 -> UGL:SM0805
- moved R1 4.16 mm to (201.6, 147.7)
- moved U4 0.28 mm to (205.9, 140.6), turned to 0 degrees
Routing:
- net GND: track 268.2 -> 286.4 mm, vias 141 -> 142
- net /SCL_BOTTOM: track 2.96 -> 9.51 mm
- net Net-(P1-Pad10): track 11.7 -> 7.13 mm
- net /RDY: track 37.9 -> 41.4 mm
- net /VCC_BOTTOM: track 16.8 -> 13.4 mm
- net /TX5: track 16.7 -> 18.0 mm
- net /SDA_BOTTOM: track 7.78 -> 6.87 mm
- net /RX3: track 9.55 -> 10.4 mm, vias 1 -> 3
- net /SDA: track 20.4 -> 19.8 mm
- net /RX2: track 11.9 -> 12.3 mm, vias 1 -> 3

Commit message: Spruce up silk screen.
Parts:
- R1: value 33 -> 0

Commit message: Bump board version to 5.0.0
Other:
- board text added: "PCB_ID: touchpad_top_5.0.0"
- board text removed: "PCB_ID: touchpad_top_4.0.0"
Changed lines of the file:
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@@
   (title_block
     (title "UHK Touchpad Module - Top Board")
-    (rev 4.0.0)
+    (rev 5.0.0)
     (company "Ultimate Gadget Laboratories Kft.")
   )
@@
   (gr_line (start 219.1766 151.1808) (end 219.1766 120.65) (layer F.Mask) (width 0.6))
   (gr_line (start 193.7512 157.7848) (end 217.8 157.7848) (layer F.Mask) (width 0.6))
-  (gr_text "PCB_ID: touchpad_top_4.0.0" (at 205.2 120.3) (layer B.SilkS)
+  (gr_text "PCB_ID: touchpad_top_5.0.0" (at 205.2 120.3) (layer B.SilkS)
     (effects (font (size 0.75 0.75) (thickness 0.15)) (justify mirror))
   )

Commit message: Bump version to 5.0.1
Other:
- board text added: "PCB_ID: touchpad_top_5.0.1"
- board text removed: "PCB_ID: touchpad_top_5.0.0"
Changed lines of the file:
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@@
   (title_block
     (title "UHK Touchpad Module - Top Board")
-    (rev 5.0.0)
+    (rev 5.0.1)
     (company "Ultimate Gadget Laboratories Kft.")
   )
@@
   (gr_line (start 219.1766 151.1808) (end 219.1766 120.65) (layer F.Mask) (width 0.6))
   (gr_line (start 193.7512 157.7848) (end 217.8 157.7848) (layer F.Mask) (width 0.6))
-  (gr_text "PCB_ID: touchpad_top_5.0.0" (at 205.2 120.3) (layer B.SilkS)
+  (gr_text "PCB_ID: touchpad_top_5.0.1" (at 205.2 120.3) (layer B.SilkS)
     (effects (font (size 0.75 0.75) (thickness 0.15)) (justify mirror))
   )

Commit message: Modified contour.
Other:
- board size 28.3 x 40 mm -> 28.4 x 40.1 mm
